File: BoardTwo/BoardTwo.kicad_sch (KiCad schematic)
At the start: 0 parts

Commit message: Added in the basic components
MCU: STM32G474RETx
LEDs
MOSFET; N-Channel Enhancement Types
Pin Header(Plugs into PCB 1)
Parts:
- added D1: RED_LED, LED_THT:LED_D5.0mm, symbol Device:LED
- added D2: GREEN_LED, LED_THT:LED_D5.0mm, symbol Device:LED
- added J1: Conn_01x04_Pin, Package_QFP:LQFP-64_10x10mm_P0.5mm, symbol Connector:Conn_01x04_Pin
- added Q1, Q2: Q_NMOS_DGS, Package_DFN_QFN:Diodes_DFN1006-3, symbol Transistor_FET:Q_NMOS_DGS
- added R1, R2: 330, Package_TO_SOT_SMD:SOT-223-3_TabPin2, symbol Device:R_US
- added U1: STM32G474RETx, Package_QFP:LQFP-64_10x10mm_P0.5mm, symbol MCU_ST_STM32G4:STM32G474RETx
Connections:
- new net: D2.2 (A), R1.1
- new net: Q1.1 (D), R1.2
- new net: U1.15 (VSS), U1.31 (VSS), U1.47 (VSS), U1.63 (VSS)
- new net: D1.2 (A), R2.1
- new net: Q2.1 (D), R2.2
